File: Kettenroboter/Hardware/KiCad/Basis/Basis.kicad_pcb (KiCad board)
At the start: 2 copper layers, 36 parts, among them J10 Screw_Terminal_01x02, J2 Screw_Terminal_01x02, J21 Screw_Terminal_01x02, J22 Screw_Terminal_01x02, J23 Screw_Terminal_01x02, J24 Screw_Terminal_01x02, J3 Screw_Terminal_01x02, J4 Screw_Terminal_01x02, J5 Screw_Terminal_01x02, J6 Screw_Terminal_01x02, J7 Screw_Terminal_01x02, J8 Screw_Terminal_01x02, J9 Screw_Terminal_01x02, Q1 BSS138, Q2 BSS138, Q3 BSS138, Q4 BSS138, Q5 NMOS, Q6 NMOS, U3 SN74LS07

Commit message: Neues Pico W Symol & Footprint
Parts:
- removed J10, J21, J22, J23, J24, J8, J9: Screw_Terminal_01x02, Library:CONN_39773-0002_MOL
- added C2: C, Capacitor_SMD:C_1206_3216Metric_Pad1.33x1.80mm_HandSolder, F.Cu at (2.50, 1.18)
- added C3: C, Capacitor_SMD:C_1206_3216Metric_Pad1.33x1.80mm_HandSolder, F.Cu at (2.50, 4.53)
- added C4: C, Capacitor_SMD:C_1206_3216Metric_Pad1.33x1.80mm_HandSolder, F.Cu at (2.50, 7.88)
- added C6: C, Capacitor_SMD:C_1206_3216Metric_Pad1.33x1.80mm_HandSolder, F.Cu at (2.50, 11.2)
- added D5: BAT46, Diode_THT:D_DO-35_SOD27_P7.62mm_Horizontal, F.Cu at (7.08, 1.27)
- added D6: BAT46, Diode_THT:D_DO-35_SOD27_P7.62mm_Horizontal, F.Cu at (7.08, 4.83)
- added D7: BAT46, Diode_THT:D_DO-35_SOD27_P7.62mm_Horizontal, F.Cu at (7.08, 8.38)
- added U2: NCP1117LPST33T3G, Library:NCP1117_SOT230P700X175-4N, F.Cu at (57.8, 48.3)
- J2, J3, J4, J5, J6, J7: value Screw_Terminal_01x02 -> 691241500008; footprint Library:CONN_39773-0002_MOL -> Library:WR-TBL_V2_691241500008
- moved J7 243.3 mm to (205.7, 256.5), turned to -90 degrees
- moved J6 204.8 mm to (205.7, 210.8), turned to -90 degrees
- moved J5 190.5 mm to (205.7, 165.1), turned to -90 degrees
- moved J2 186.9 mm to (203.2, 33.0), turned to -90 degrees
- moved J4 180.4 mm to (203.2, 119.4), turned to -90 degrees
- moved J3 180.3 mm to (203.2, 76.2), turned to -90 degrees
- moved U1 21.5 mm to (124.5, 33.0)
Connections:
- net VSYS renamed /VSYS
- D2 pad 1: +3V3 -> /+3V3
- J2 pad 1: ADC0 -> /+3V3
- J2 pad 2: ADC1 -> ADC0
- J3 pad 1: ADC2 -> QEI0_A
- J3 pad 2: ADC_GND -> QEI0_B
- J4 pad 1: QEI0_A -> /+3V3
- J4 pad 2: QEI0_B -> HALL0
- J5 pad 1: QEI1_A -> I2C0 - HV
- J5 pad 2: QEI1_B -> I2C0 -SDA - HV
- J6 pad 1: HALL0 -> D_out_12
- J6 pad 2: HALL1 -> GND
- J7 pad 1: I2C0 -SDA - HV -> BRAKE0 -
- J7 pad 2: I2C0 - SCL - HV -> BRAKE1 -
- Q1 pad 1: +3V3 -> /+3V3
- Q2 pad 1: +3V3 -> /+3V3
- Q3 pad 1: +3V3 -> /+3V3
- Q4 pad 1: +3V3 -> /+3V3
- R1 pad 1: +3V3 -> /+3V3
- R11 pad 1: ADC2_uf -> Net-(D5-K)
- R11 pad 2: ADC2 -> Net-(J11-Pin_1)
- R2 pad 1: unconnected-(R2-Pad1) -> Net-(J16-Pin_2)
- R3 pad 1: +3V3 -> /+3V3
- R4 pad 1: unconnected-(R4-Pad1) -> Net-(J16-Pin_2)
- R5 pad 1: +3V3 -> /+3V3
- R6 pad 1: unconnected-(R6-Pad1) -> Net-(J17-Pin_2)
- R7 pad 1: +3V3 -> /+3V3
- R8 pad 1: unconnected-(R8-Pad1) -> Net-(J17-Pin_2)
- U3 pad 1: GPO10 -> Net-(J11-Pin_3)
- U3 pad 10: D4 -> D_out_12
- U3 pad 11: GPO14 -> Net-(J13-Pin_3)
- U3 pad 12: D5 -> D_out_12
- U3 pad 13: GPO15 -> Net-(J13-Pin_3)
- U3 pad 2: D0 -> D_out_10
- U3 pad 3: GPO11 -> Net-(J11-Pin_3)
- U3 pad 4: D1 -> D_out_10
- U3 pad 5: GPO12 -> Net-(J12-Pin_3)
- U3 pad 6: D2 -> D_out_11
- U3 pad 8: D3 -> D_out_11
- U3 pad 9: GPO13 -> Net-(J12-Pin_3)

Commit message: pcb layout fnished
Parts:
- removed U1: ~, Library:Raspberrypi pico2 THT
- added +12V1: TestPoint, TestPoint:TestPoint_Pad_D2.5mm, F.Cu at (106.7, 84.8)
- added +3V3: TestPoint, TestPoint:TestPoint_Pad_D2.5mm, F.Cu at (155.1, 45.8)
- added A1: RaspberryPi_Pico_W, Module:RaspberryPi_Pico_Common_THT, F.Cu at (129.7, 39.5)
- added C11: C, Capacitor_SMD:C_1206_3216Metric_Pad1.33x1.80mm_HandSolder, F.Cu at (111.5, 117.5)
- added C12: C, Capacitor_SMD:C_1206_3216Metric_Pad1.33x1.80mm_HandSolder, F.Cu at (116.6, 109.6)
- added C13: C, Capacitor_SMD:C_1206_3216Metric_Pad1.33x1.80mm_HandSolder, F.Cu at (112.8, 102.0)
- added C14: 470u, Capacitor_THT:CP_Radial_D5.0mm_P2.50mm, F.Cu at (96.1, 40.9)
- added C15: 10n, Capacitor_SMD:C_1206_3216Metric_Pad1.33x1.80mm_HandSolder, F.Cu at (103.3, 42.3)
- added D10: BAT46, Diode_THT:D_DO-35_SOD27_P7.62mm_Horizontal, F.Cu at (112.8, 94.9)
- added D3: D, Diode_THT:D_5KPW_P7.62mm_Vertical_AnodeUp, F.Cu at (155.2, 117.8)
- added D4: D, Diode_THT:D_5KPW_P7.62mm_Vertical_AnodeUp, F.Cu at (163.8, 121.4)
- added D8: 1N5817, Diode_THT:D_DO-41_SOD81_P10.16mm_Horizontal, B.Cu at (153.7, 49.5)
- added D9: BAT46, Diode_THT:D_DO-35_SOD27_P7.62mm_Horizontal, F.Cu at (116.1, 97.0)
- added GND1: TestPoint, TestPoint:TestPoint_Pad_D2.5mm, F.Cu at (106.6, 89.7)
- added GND2: TestPoint, TestPoint:TestPoint_Pad_D2.5mm, F.Cu at (156.6, 50.0)
- added GND3: TestPoint, TestPoint:TestPoint_Pad_D2.5mm, F.Cu at (124.2, 52.6)
- added H1: MountingHole_Pad, MountingHole:MountingHole_3.2mm_M3_Pad_Via, F.Cu at (118.3, 46.0)
- added H2: MountingHole_Pad, MountingHole:MountingHole_3.2mm_M3_Pad_Via, F.Cu at (101.1, 75.3)
- added H3: MountingHole_Pad, MountingHole:MountingHole_4.3mm_M4_Pad_Via, F.Cu at (93.6, 48.4)
- added H4: MountingHole_Pad, MountingHole:MountingHole_4.3mm_M4_Pad_Via, F.Cu at (143.4, 96.7)
- added H5: MountingHole_Pad, MountingHole:MountingHole_4.3mm_M4_Pad_Via, F.Cu at (131.2, 123.4)
- added H6: MountingHole_Pad, MountingHole:MountingHole_4.3mm_M4_Pad_Via, F.Cu at (169.7, 130.2)
- added J1: 691103110002, Library:WR-TBL_V3_2pin_691103110002, F.Cu at (172.6, 42.7)
- added J10: 691103110002, Library:WR-TBL_V3_2pin_691103110002, F.Cu at (172.6, 98.4)
- added J11: Conn_01x03, Connector_PinHeader_2.54mm:PinHeader_1x03_P2.54mm_Vertical, F.Cu at (120.4, 113.9)
- added J12: Conn_01x03, Connector_PinHeader_2.54mm:PinHeader_1x03_P2.54mm_Vertical, F.Cu at (120.1, 106.4)
- added J13: Conn_01x03, Connector_PinHeader_2.54mm:PinHeader_1x03_P2.54mm_Vertical, F.Cu at (120.3, 99.4)
- added J14: Conn_01x03, Connector_PinHeader_2.54mm:PinHeader_1x03_P2.54mm_Vertical, F.Cu at (117.1, 132.0)
- added J15: Conn_01x01, Connector_PinHeader_2.54mm:PinHeader_1x01_P2.54mm_Vertical, F.Cu at (120.7, 129.4)
- added J16: Conn_01x03, Connector_PinHeader_2.54mm:PinHeader_1x03_P2.54mm_Vertical, F.Cu at (155.7, 77.5)
- added J17: Conn_01x03, Connector_PinHeader_2.54mm:PinHeader_1x03_P2.54mm_Vertical, F.Cu at (156.0, 92.1)
- added J18: 691103110002, Library:WR-TBL_V3_2pin_691103110002, F.Cu at (172.6, 77.1)
- added J19: 691103110002, Library:WR-TBL_V3_2pin_691103110002, F.Cu at (172.6, 84.2)
- added J20: 691103110002, Library:WR-TBL_V3_2pin_691103110002, F.Cu at (92.8, 130.9)
- added J21: 691103110002, Library:WR-TBL_V3_2pin_691103110002, F.Cu at (92.8, 123.8)
- added J22: 691103110002, Library:WR-TBL_V3_2pin_691103110002, F.Cu at (92.8, 116.7)
- added J23: 691103110002, Library:WR-TBL_V3_2pin_691103110002, F.Cu at (92.8, 109.6)
- added J24: 691103110002, Library:WR-TBL_V3_2pin_691103110002, F.Cu at (92.8, 102.5)
- added J25: 691103110002, Library:WR-TBL_V3_2pin_691103110002, F.Cu at (172.6, 108.1)
- added J26: 691103110002, Library:WR-TBL_V3_2pin_691103110002, F.Cu at (172.6, 115.2)
- added J27: 691103110002, Library:WR-TBL_V3_2pin_691103110002, F.Cu at (92.8, 88.5)
- added J8: 691103110002, Library:WR-TBL_V3_2pin_691103110002, F.Cu at (172.6, 67.4)
- added J9: 691103110002, Library:WR-TBL_V3_2pin_691103110002, F.Cu at (172.6, 91.3)
- added R14: R, Resistor_SMD:R_1206_3216Metric_Pad1.30x1.75mm_HandSolder, F.Cu at (108.8, 117.5)
- added R15: R, Resistor_SMD:R_1206_3216Metric_Pad1.30x1.75mm_HandSolder, F.Cu at (109.2, 108.1)
- added R16: R, Resistor_SMD:R_1206_3216Metric_Pad1.30x1.75mm_HandSolder, F.Cu at (113.8, 109.6)
- added R17: R, Resistor_SMD:R_1206_3216Metric_Pad1.30x1.75mm_HandSolder, F.Cu at (106.0, 100.4)
- added R18: R, Resistor_SMD:R_1206_3216Metric_Pad1.30x1.75mm_HandSolder, F.Cu at (110.2, 102.0)
- added R19: R, Resistor_SMD:R_1206_3216Metric_Pad1.30x1.75mm_HandSolder, F.Cu at (97.9, 119.5)
- added R20: R, Resistor_SMD:R_1206_3216Metric_Pad1.30x1.75mm_HandSolder, F.Cu at (110.6, 127.0)
- added R21: R, Resistor_SMD:R_1206_3216Metric_Pad1.30x1.75mm_HandSolder, F.Cu at (112.3, 130.9)
- added VBUS1: TestPoint, TestPoint:TestPoint_Pad_D2.5mm, F.Cu at (161.3, 39.9)
- added VSYS1: TestPoint, TestPoint:TestPoint_Pad_D2.5mm, F.Cu at (124.3, 40.9)
- added buck_converter_ph_(12to5)1: ~, Library:BA_Buck_mangled_PH, F.Cu at (98.3, 82.4)
- D1, U2: moved to B.Cu
- D2: value 1N5817 -> BAT46; footprint Diode_THT:D_DO-41_SOD81_P10.16mm_Horizontal -> Diode_THT:D_DO-35_SOD27_P7.62mm_Horizontal; moved to B.Cu
- J2, J3, J4, J5, J6, J7: value 691241500008 -> 691103110002; footprint Library:WR-TBL_V2_691241500008 -> Library:WR-TBL_V3_2pin_691103110002
- moved J7 199.1 mm to (172.6, 60.2)
- moved C3 169.8 mm to (167.3, 45.7), turned to -90 degrees
- moved C6 169.6 mm to (167.3, 51.7), turned to 90 degrees
- moved C2 165.5 mm to (161.5, 46.8), turned to -90 degrees
- moved C4 165.2 mm to (161.7, 52.0), turned to 90 degrees
- moved D5 150.5 mm to (100.9, 118.9), turned to 100 degrees
- moved D6 145.6 mm to (105.4, 112.2), turned to 135 degrees
- moved D7 137.2 mm to (105.8, 103.6), turned to 180 degrees
- moved R9 129.1 mm to (164.5, 45.6), turned to 90 degrees
- moved R10 128.4 mm to (164.5, 51.7), turned to -90 degrees
- moved D2 118.4 mm to (118.1, 121.7), turned to 180 degrees
- moved R13 107.0 mm to (145.9, 115.4)
- moved R12 106.7 mm to (145.9, 110.5)
- moved U2 97.3 mm to (154.9, 42.0)
- moved D1 93.0 mm to (134.7, 44.5), turned to 180 degrees
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Connections:
- J2 pad 1: /+3V3 -> ADC1
- J2 pad 2: ADC0 -> /ADC_GND
- J4 pad 1: /+3V3 -> QEI1_A
- J4 pad 2: HALL0 -> QEI1_B
- J5 pad 1: I2C0 - HV -> QEI2_A
- J5 pad 2: I2C0 -SDA - HV -> QEI2_B
- J6 pad 1: D_out_12 -> QEI3_A
- J6 pad 2: GND -> QEI3_B
- J7 pad 1: BRAKE0 - -> /+3V3
- J7 pad 2: BRAKE1 - -> HALL0
- Q4 pad 3: I2C1 - SDA - HV -> I2C1 - SCL - HV
- R11 pad 2: Net-(J11-Pin_1) -> Net-(D2-A)
- R8 pad 2: I2C1 - SDA - HV -> I2C1 - SCL - HV
- U3 pad 14: GPO_Vcc -> GND
- U3 pad 7: GND -> /VBUS
Routing:
- net /+3V3: track 0.00 -> 315.9 mm, vias 0 -> 11
- net /VSYS: track 0.00 -> 207.6 mm, vias 0 -> 3
- net /+12V: track 0.00 -> 172.1 mm
- net /VBUS: track 0.00 -> 139.4 mm, vias 0 -> 3
- net QEI0_A: track 0.00 -> 80.0 mm
- net QEI0_B: track 0.00 -> 77.2 mm
- net QEI1_A: track 0.00 -> 75.5 mm
- net I2C1 - SCL: track 0.00 -> 75.4 mm
- net I2C0 - SCL: track 0.00 -> 73.0 mm
- net GPIO12: track 0.00 -> 72.2 mm
- net QEI1_B: track 0.00 -> 71.2 mm
- net I2C1 - SDA: track 0.00 -> 70.9 mm
- net QEI2_A: track 0.00 -> 69.6 mm
- net QEI2_B: track 0.00 -> 67.6 mm
- net GPIO11: track 0.00 -> 67.1 mm
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- added copper zone on F.Cu, net /+12V
- added copper zone on B.Cu, net /+3V3
- added copper zone on B.Cu, net /ADC_GND
- added copper zone on F.Cu, net /ADC_GND
- added copper zone on B.Cu, net GND
- added copper zone on F.Cu, net GND
Other:
- board outline added: 90.6 x 101.2 mm

Commit message: Fast finale Version
Nach Crash gefixt
Parts:
- added C1: 10u, Capacitor_SMD:C_1206_3216Metric_Pad1.33x1.80mm_HandSolder, B.Cu at (144.0, 40.7)
- added C10: C_Polarized, Capacitor_THT:CP_Radial_D5.0mm_P2.50mm, F.Cu at (157.1, 99.5)
- added C16: 10n, Capacitor_SMD:C_1206_3216Metric_Pad1.33x1.80mm_HandSolder, F.Cu at (111.6, 119.8)
- added C5: 10u, Capacitor_SMD:C_1206_3216Metric_Pad1.33x1.80mm_HandSolder, B.Cu at (167.6, 41.1)
- added C7: C_Polarized, Capacitor_THT:CP_Radial_D5.0mm_P2.50mm, F.Cu at (162.8, 40.0)
- added C8: C_Polarized, Capacitor_THT:CP_Radial_D5.0mm_P2.50mm, F.Cu at (128.4, 116.0)
- added C9: C_Polarized, Capacitor_THT:CP_Radial_D5.0mm_P2.50mm, F.Cu at (166.6, 69.0)
- added J28: Conn_01x02, Connector_PinHeader_2.54mm:PinHeader_1x02_P2.54mm_Vertical, F.Cu at (153.8, 62.4)
- added R23: R, Resistor_SMD:R_1206_3216Metric_Pad1.30x1.75mm_HandSolder, B.Cu at (136.4, 127.6)
- added R25: R, Resistor_SMD:R_1206_3216Metric_Pad1.30x1.75mm_HandSolder, B.Cu at (139.2, 124.8)
- added R27: R, Resistor_SMD:R_1206_3216Metric_Pad1.30x1.75mm_HandSolder, B.Cu at (142.5, 127.5)
- added R29: R, Resistor_SMD:R_1206_3216Metric_Pad1.30x1.75mm_HandSolder, B.Cu at (146.1, 124.8)
- added R31: R, Resistor_SMD:R_1206_3216Metric_Pad1.30x1.75mm_HandSolder, B.Cu at (160.4, 124.8)
- added R33: R, Resistor_SMD:R_1206_3216Metric_Pad1.30x1.75mm_HandSolder, B.Cu at (149.7, 127.5)
- added R35: R, Resistor_SMD:R_1206_3216Metric_Pad1.30x1.75mm_HandSolder, B.Cu at (153.3, 124.8)
- added R37: R, Resistor_SMD:R_1206_3216Metric_Pad1.30x1.75mm_HandSolder, B.Cu at (157.0, 127.4)
- D2: moved to F.Cu
- moved J11 23.7 mm to (103.9, 96.9), turned to 180 degrees
- moved J12 14.9 mm to (108.7, 96.9), turned to 180 degrees
- moved D10 14.6 mm to (125.6, 101.9)
- moved D9 13.9 mm to (125.7, 107.1), turned to 180 degrees
- moved R19 12.9 mm to (100.7, 132.1), turned to 180 degrees
- moved D2 11.6 mm to (125.7, 112.9)
- moved R20 9.75 mm to (101.0, 128.4)
- moved VBUS1 9.45 mm to (151.9, 38.9)
- moved +12V1 7.63 mm to (99.1, 85.2), turned to -90 degrees
- moved D5 7.60 mm to (105.8, 113.2), turned to 180 degrees
- moved GND1 7.51 mm to (99.1, 89.2), turned to -90 degrees
- moved J13 7.48 mm to (113.3, 96.8), turned to 180 degrees
- moved J14 7.45 mm to (122.3, 126.6), turned to 0 degrees
- moved R11 6.48 mm to (109.3, 114.3), turned to -90 degrees
- moved R21 6.23 mm to (114.0, 125.0)
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Connections:
- A1 pad 33: /ADC_GND -> GND
- C2 pad 2: /ADC_GND -> GND
- C3 pad 2: /ADC_GND -> GND
- C4 pad 2: /ADC_GND -> GND
- C6 pad 2: /ADC_GND -> GND
- J11 pad 2: GPIO12 -> GPIO10
- J13 pad 2: GPIO10 -> GPIO12
- J16 pad 1: /VBUS -> /VSYS
- J17 pad 1: /VBUS -> /VSYS
- J18 pad 2: I2C0 -SDA - HV -> I2C0 - SDA - HV
- J2 pad 2: /ADC_GND -> GND
- J20 pad 1: V_D_out_ext -> GND
- J20 pad 2: GND -> V_D_out_ext
- J25 pad 1: GND -> /PWR-GND
- Q5 pad 3: GND -> /PWR-GND
- Q6 pad 3: GND -> /PWR-GND
- U3 pad 14: GND -> /VSYS
- U3 pad 7: /VBUS -> GND
Routing:
- net /VSYS: track 207.6 -> 379.0 mm, vias 3 -> 11
- net /VBUS: track 139.4 -> 6.45 mm, vias 3 -> 0
- net GPIO12: track 72.2 -> 52.0 mm
- net Net-(J12-Pin_3): track 44.4 -> 62.1 mm, vias 1 -> 4
- net /+3V3: track 315.9 -> 300.5 mm
- net Net-(D2-A): track 19.2 -> 34.4 mm
- net Net-(D9-A): track 13.1 -> 26.7 mm
- net Net-(J11-Pin_3): track 25.1 -> 38.2 mm, vias 2 -> 0
- net D_out_11: track 16.5 -> 28.2 mm, vias 2 -> 0
- net GND: track 15.3 -> 5.76 mm, vias 22 -> 55
- net GPIO11: track 67.1 -> 57.8 mm
- net D_out_12: track 33.6 -> 25.1 mm
- net QEI3_A: track 65.9 -> 73.3 mm, vias 0 -> 1
- net RUN: track 0.00 -> 7.38 mm
- net D_out_10: track 24.8 -> 32.1 mm
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- removed copper zone on B.Cu, net /ADC_GND
- removed copper zone on F.Cu, net /ADC_GND

Commit message: final final final
Parts:
- added C17: 10n, Capacitor_SMD:C_1206_3216Metric_Pad1.33x1.80mm_HandSolder, F.Cu at (127.1, 104.4)
- added C18: 10n, Capacitor_SMD:C_1206_3216Metric_Pad1.33x1.80mm_HandSolder, F.Cu at (174.9, 123.4)
- added C19: 10n, Capacitor_SMD:C_1206_3216Metric_Pad1.33x1.80mm_HandSolder, F.Cu at (160.1, 67.2)
- added C20: 10n, Capacitor_SMD:C_1206_3216Metric_Pad1.33x1.80mm_HandSolder, F.Cu at (127.4, 110.0)
- added D11: 1N5817, Diode_THT:D_DO-41_SOD81_P10.16mm_Horizontal, F.Cu at (92.8, 82.3)
- D1: moved to F.Cu
- D8: value 1N5817 -> BAT46; footprint Diode_THT:D_DO-41_SOD81_P10.16mm_Horizontal -> Diode_THT:D_DO-35_SOD27_P7.62mm_Horizontal
- moved GND2 53.5 mm to (117.7, 86.9)
- moved GND3 33.2 mm to (157.4, 50.7)
- moved VSYS1 31.9 mm to (156.2, 39.1)
- moved D1 10.6 mm to (124.7, 41.0), turned to -90 degrees
- moved D8 5.30 mm to (157.9, 46.3), turned to -145 degrees
- moved GND1 2.69 mm to (99.4, 91.8), turned to 0 degrees
- moved C1 2.36 mm to (144.0, 43.1)
- moved +12V1 1.42 mm to (99.3, 86.6), turned to 0 degrees
- moved +3V3 1.17 mm to (154.2, 45.1)
- moved J15 0.76 mm to (125.1, 129.2)
- moved J14 0.13 mm to (122.4, 126.6)
Connections:
- C1 pad 1: /VBUS -> /VSYS
- H1 pad 1: GND -> unconnected-(H1-Pad1)
- H2 pad 1: GND -> unconnected-(H2-Pad1)
- H3 pad 1: GND -> unconnected-(H3-Pad1)
- H4 pad 1: GND -> unconnected-(H4-Pad1)
- H5 pad 1: GND -> unconnected-(H5-Pad1)
- H6 pad 1: GND -> unconnected-(H6-Pad1)
- J20 pad 1: GND -> V_D_out_ext
- J20 pad 2: V_D_out_ext -> GND
- J25 pad 1: /PWR-GND -> GND
- J27 pad 2: /+12V -> Net-(D11-K)
- Q1 pad 3: I2C0 -SDA - HV -> I2C0 - SDA - HV
- Q5 pad 3: /PWR-GND -> GND
- Q6 pad 3: /PWR-GND -> GND
- R2 pad 2: I2C0 -SDA - HV -> I2C0 - SDA - HV
- U2 pad 3: /VBUS -> /VSYS
Routing:
- net /+3V3: track 300.5 -> 322.7 mm, vias 11 -> 13
- net I2C0 -SDA - HV: track 12.7 -> 0.00 mm
- net I2C0 - SDA - HV: track 0.00 -> 12.7 mm
- net GND: track 5.76 -> 15.5 mm, vias 55 -> 137
- net Net-(D11-K): track 0.00 -> 4.47 mm
- net Net-(D1-A): track 44.3 -> 40.1 mm
- net D_out_12: track 25.1 -> 28.0 mm
- net /+12V: track 172.1 -> 173.5 mm
- net /VBUS: track 6.45 -> 5.62 mm
- net Net-(A1-3V3): track 3.99 -> 4.70 mm
- net /VSYS: track 379.0 -> 378.3 mm, vias 11 -> 10
- removed copper zone on B.Cu, net /+3V3
Other:
- board size 90.6 x 101.2 mm -> 90.6 x 102.2 mm
- board text added: "+12V|Brake1|Brake0|GND"
- board text added: "+12V|GND"
- board text added: "+5V"
- board text added: "10"
- board text added: "11"
- board text added: "12"
- board text added: "GND|ADC1|ADC0|+3V3"
- board text added: "GND|HALL1|HALL0|+3V3"
- board text added: "GND|SCL0|SDA0|0_V_ex"
- board text added: "GND|SCL1|SDA1|1_V_ex"
- board text added: "GND|Vout_ex"
- board text added: "GPIO"
- board text added: "I2C0"
- board text added: "I2C1"
- board text added: "INPUT"
- board text added: "N.C. |DI12|DI11|DI10"
- board text added: "OUTPUT"
- board text added: "QEI1A|QEI1B|"
- board text added: "QEI2A|QEI2B|"
- board text added: "QEI3A|QEI3B|"
- board text added: "V_ex"
- board text added: "|GND|DO12|DO11|DO10|"
- board text added: "|QEI0A|QEI0B|"

Commit message: _
Other:
- board text added: "3V3"
- board text added: "5V"
- board text added: "V_ext"
- board text added: "Vcc_DO"
Changed lines of the file:
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@@
 		(tags "Through hole pin header THT 1x03 2.54mm single row")
 		(property "Reference" "J14"
-			(at 0 -2.38 0)
+			(at 2.54 8.509 0)
 			(layer "F.SilkS")
 			(effects
@@
 		(tags "Through hole pin header THT 1x01 2.54mm single row")
 		(property "Reference" "J15"
-			(at 0 -2.38 90)
+			(at 5.715 -2.286 90)
 			(layer "F.SilkS")
 			(effects
@@
 		(tags "resistor handsolder")
 		(property "Reference" "R23"
-			(at 4.191 -0.889 0)
+			(at 4.064 -1.397 0)
 			(layer "B.SilkS")
 			(effects
@@
 		)
 	)
+	(gr_text "5V"
+		(at 122.555 124.079 0)
+		(layer "F.SilkS")
+		(effects
+			(font
+				(size 0.65 0.75)
+				(thickness 0.15)
+			)
+		)
+	)
 	(gr_text "+5V"
 		(at 149.225 78.359 0)
@@
 		)
 	)
+	(gr_text "Vcc_DO"
+		(at 118.745 129.286 0)
+		(layer "F.SilkS")
+		(effects
+			(font
+				(size 0.65 0.75)
+				(thickness 0.15)
+			)
+		)
+	)
 	(gr_text "INPUT"
 		(at 114.935 92.837 0)
@@
 		)
 	)
+	(gr_text "V_ext"
+		(at 118.999 132.08 0)
+		(layer "F.SilkS")
+		(effects
+			(font
+				(size 0.65 0.75)
+				(thickness 0.15)
+			)
+		)
+	)
 	(gr_text "|QEI0A|QEI0B|"
 		(at 136.271 137.287 0)
@@
 		)
 	)
+	(gr_text "3V3"
+		(at 127.762 129.54 0)
+		(layer "F.SilkS")
+		(effects
+			(font
+				(size 0.65 0.75)
+				(thickness 0.15)
+			)
+		)
+	)
 	(gr_text "V_ex"
 		(at 149.352 73.025 0)
@@
 	(dimension
 		(type orthogonal)
-		(layer "Dwgs.User")
+		(layer "F.SilkS")
 		(pts
-			(xy 177.673 138.049) (xy 87.122 138.049)
+			(xy 87.122 138.049) (xy 177.673 138.049)
 		)
-		(height 13.462)
+		(height 16.764)
 		(orientation 0)
 		(format
@@
 		)
 		(style
-			(thickness 0.2)
+			(thickness 0.1)
 			(arrow_length 1.27)
 			(text_position_mode 0)
@@
 		)
 		(gr_text "90,551"
-			(at 132.3975 149.711 0)
-			(layer "Dwgs.User")
+			(at 132.3975 153.713 0)
+			(layer "F.SilkS")
 			(effects
 				(font
-					(size 1.5 1.5)
-					(thickness 0.3)
+					(size 1 1)
+					(thickness 0.1)
 				)
 			)
@@
 	(dimension
 		(type orthogonal)
-		(layer "Dwgs.User")
+		(layer "F.SilkS")
 		(pts
-			(xy 177.673 138.049) (xy 177.673 36.83)
+			(xy 177.673 35.814) (xy 177.673 138.049)
 		)
-		(height 16.51)
+		(height 21.336)
 		(orientation 1)
 		(format
@@
 		)
 		(style
-			(thickness 0.2)
+			(thickness 0.1)
 			(arrow_length 1.27)
 			(text_position_mode 0)
@@
 			(keep_text_aligned yes)
 		)
-		(gr_text "101,219"
-			(at 192.383 87.4395 90)
-			(layer "Dwgs.User")
+		(gr_text "102,235"
+			(at 197.909 86.9315 90)
+			(layer "F.SilkS")
 			(effects
 				(font
-					(size 1.5 1.5)
-					(thickness 0.3)
+					(size 1 1)
+					(thickness 0.1)
 				)
-				(justify mirror)
 			)
 		)

Commit message: All Parts placed (BOM)
Parts:
- C11, C12, C13, C2, C4: value C -> 1n
- R10, R9: value R -> 720
- R11, R15, R17, R19, R20, R21: value R -> 1k
- R12: value R -> 1,3K
- R13: value R -> 1.3k
- R14, R16, R18: value R -> 10k
Changed lines of the file:
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@@
 			)
 		)
-		(property "Value" "R"
+		(property "Value" "10k"
 			(at 0 1.83 90)
 			(layer "F.Fab")
@@
 			)
 		)
-		(property "Value" "R"
+		(property "Value" "10k"
 			(at 0 1.83 90)
 			(layer "F.Fab")
@@
 			)
 		)
-		(property "Value" "R"
+		(property "Value" "1k"
 			(at 0 1.83 90)
 			(layer "F.Fab")
@@
 			)
 		)
-		(property "Value" "C"
+		(property "Value" "1n"
 			(at 0 1.85 90)
 			(layer "F.Fab")
@@
 			)
 		)
-		(property "Value" "R"
+		(property "Value" "10k"
 			(at 0 1.83 90)
 			(layer "F.Fab")
@@
 			)
 		)
-		(property "Value" "C"
+		(property "Value" "1n"
 			(at 0 1.85 90)
 			(layer "F.Fab")
@@
 			)
 		)
-		(property "Value" "R"
+		(property "Value" "1k"
 			(at 0 1.83 90)
 			(layer "F.Fab")
@@
 			)
 		)
-		(property "Value" "R"
+		(property "Value" "1k"
 			(at 0 1.83 0)
 			(layer "F.Fab")
@@
 			)
 		)
-		(property "Value" "R"
+		(property "Value" "1k"
 			(at 0 1.83 0)
 			(layer "F.Fab")
@@
 			)
 		)
-		(property "Value" "R"
+		(property "Value" "720"
 			(at 0 0 90)
 			(layer "F.Fab")
@@
 			)
 		)
-		(property "Value" "R"
+		(property "Value" "1k"
 			(at 0 1.83 90)
 			(layer "F.Fab")
@@
 			)
 		)
-		(property "Value" "C"
+		(property "Value" "1n"
 			(at 0 0 90)
 			(layer "F.Fab")
@@
 			)
 		)
-		(property "Value" "C"
+		(property "Value" "1n"
 			(at 0 1.85 90)
 			(layer "F.Fab")
@@
 			)
 		)
-		(property "Value" "C"
+		(property "Value" "1n"
 			(at 0 1.85 90)
 			(layer "F.Fab")
@@
 			)
 		)
-		(property "Value" "R"
+		(property "Value" "1.3k"
 			(at 0 1.83 0)
 			(layer "F.Fab")
@@
 			)
 		)
-		(property "Value" "R"
+		(property "Value" "1k"
 			(at 0 2.54 90)
 			(layer "F.Fab")
@@
 			)
 		)
-		(property "Value" "R"
+		(property "Value" "1,3K"
 			(at 0 1.83 0)
 			(layer "F.Fab")
@@
 			)
 		)
-		(property "Value" "R"
+		(property "Value" "720"
 			(at 0 0 90)
 			(layer "F.Fab")
